File: greenpill-f411.kicad_pcb (KiCad board)
At the start: 4 copper layers, 20.7 x 51.3 mm, 47 parts, among them J1 USB_C_Receptacle_USB2.0, J5 GPIO, J6 GPIO, J7 ST-LINK, SW1 SW_Push, SW2 SW_Push, SW3 SW_Push, U1 SPX3819M5-L-3-3, U2 W25Q32JVSS, U6 STM32F411CEUx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

Commit message: Finished
Parts:
- moved kibuzzard-63FDC36C 0.66 mm to (145.7, 94.0), turned to -90 degrees
- moved kibuzzard-63FDC37C 0.66 mm to (154.6, 94.0), turned to -90 degrees
Routing:
- net /PA4: track 19.7 -> 37.4 mm, vias 0 -> 1
- net /MEM_MISO: track 20.9 -> 36.3 mm, vias 0 -> 1
- net GND: track 14.8 -> 23.6 mm, vias 10 -> 52
- net +3V3: track 37.5 -> 39.9 mm, vias 3 -> 6
- net VCC: track 60.2 -> 59.3 mm
